File: MakerPlayground_TinyBaseBoard.sch (KiCad schematic (older format))
At the start: 43 parts, among them J1 BattCon, J2 USB, J3 D1, J4 D2, J5 I2C, J6 Analog, Q1 Q_NPN_BEC, Q2 Q_NPN_BEC, U1 MCP73831-2-OT, U2 ESP8266-12F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

Commit message: Add on-off button, I2C pullup resistor and update pcb layout
Parts:
- removed C4: 0.1uF, Capacitor_SMD:C_0603_1608Metric, symbol Device:C_Small
- removed D4: RSX101VA-30, Diode_SMD:D_TUMD2, symbol Device:D_Schottky
- added C11: 22uF, Capacitor_Tantalum_SMD:CP_EIA-3216-10_Kemet-I, symbol Device:CP1
- added R16, R17: 10K, Resistor_SMD:R_0603_1608Metric, symbol Device:R_Small
- added SW1: JS102011JCQN, GiraffeTech-Electromechanical:SW_SPDT_CK-JS102011JCQN, symbol Switch:SW_SPDT
- C3: value 10uF -> 4.7uF; footprint Capacitor_SMD:C_0805_2012Metric -> Capacitor_SMD:C_0603_1608Metric
- Q1, Q2: value Q_NPN_BEC -> MMBT2222A
- U4: value LD56100DPU33R -> LD56100; footprint GiraffeTech-ST:LD56100_DFN-8-1.6x1.2mm_P0.4 -> GiraffeTech-ST:ST_DFN-8-1EP_1.6x1.2mm_P0.4mm
Connections:
- net labels added: LDO_EN
- net labels removed: VDD
- wire segments 174 -> 180
Other:
- moved on the sheet: C10, C7, D2, D3, R6
